Commit message: Robot spawn at top of slope but urdf joints not connected properly

File: urdf/pady_simplified.urdf (robot description, URDF)
Before this commit: robot pady, 7 links, 6 joints
Joints:
- joint foot_joint_right: axis (none) -> 0 1 0; limit (none) -> lower=-0.5 upper=0.5 effort=0 velocity=5.0; type fixed -> revolute
- joint hip_joint_right: origin xyz=0 -0.10786 -0.017 rpy=0 0 0 -> xyz=0 -0.12 -0.02 rpy=0 0 0
- joint knee_joint_right: origin xyz=0 0 -0.500 rpy=0 0 0 -> xyz=0 0 -0.45 rpy=0 0 0

Commit message: Robot orientation fixed, spawns and lands at top of ramp

File: urdf/pady_simplified.urdf (robot description, URDF)
Before this commit: robot pady, 7 links, 6 joints
Joints:
- joint foot_joint_right: axis 0 1 0 -> (none); limit lower=-0.5 upper=0.5 effort=0 velocity=5.0 -> (none); type revolute -> fixed
- joint hip_joint_right: origin xyz=0 -0.12 -0.02 rpy=0 0 0 -> xyz=0 -0.10786 -0.017 rpy=0 0 0
- joint knee_joint_right: origin xyz=0 0 -0.45 rpy=0 0 0 -> xyz=0 0 -0.500 rpy=0 0 0
