Commit message: updates and fixes for sim on mini pc

File: urdf/pady.urdf (robot description, URDF)
Before this commit: robot pady, 8 links, 7 joints
Links:
- removed link world
- link base_link: geometry collision mesh filename=package://pady_robot/meshes/visual/base_link.stl scale=0.001 0.001 0.001; visual mesh filename=package://pady_robot/meshes/visual/base_link.stl scale=0.001 0.001 0.001
- link foot_left: geometry collision mesh filename=package://pady_robot/meshes/visual/left_foot.stl scale=0.001 0.001 0.001; visual mesh filename=package://pady_robot/meshes/visual/left_foot.stl scale=0.001 0.001 0.001
- link foot_right: geometry collision mesh filename=package://pady_robot/meshes/visual/right_foot.stl scale=0.001 0.001 0.001; visual mesh filename=package://pady_robot/meshes/visual/right_foot.stl scale=0.001 0.001 0.001
- link shin_left: geometry collision mesh filename=package://pady_robot/meshes/visual/shin_left.stl scale=0.001 0.001 0.001; visual mesh filename=package://pady_robot/meshes/visual/shin_left.stl scale=0.001 0.001 0.001
- link shin_right: geometry collision mesh filename=package://pady_robot/meshes/visual/shin_right.stl scale=0.001 0.001 0.001; visual mesh filename=package://pady_robot/meshes/visual/shin_right.stl scale=0.001 0.001 0.001
- link thigh_left: geometry collision mesh filename=package://pady_robot/meshes/visual/thigh_left.stl scale=0.001 0.001 0.001; visual mesh filename=package://pady_robot/meshes/visual/thigh_left.stl scale=0.001 0.001 0.001
- link thigh_right: geometry collision mesh filename=package://pady_robot/meshes/visual/thigh_right.stl scale=0.001 0.001 0.001; visual mesh filename=package://pady_robot/meshes/visual/thigh_right.stl scale=0.001 0.001 0.001
Joints:
- removed joint world_to_base

Commit message: robot walking 4 steps, yaw induces imbalance and falling. Get video no arms walk then continue to counterswing arms which will solve yaw issue.

File: urdf/pady.urdf (robot description, URDF)
Before this commit: robot pady, 7 links, 6 joints
Links:
- link foot_left: geometry collision cylinder length=0.20 radius=0.035; collision cylinder length=0.20 radius=0.035
- link foot_right: geometry collision cylinder length=0.20 radius=0.035; collision cylinder length=0.20 radius=0.035
Joints:
- joint foot_joint_left: origin xyz=0.020 0 -0.500 rpy=0 0 0 -> xyz=0.020 0 -0.500 rpy=0.05 0.0 0.0
- joint foot_joint_right: origin xyz=0.020 0 -0.500 rpy=0 0 0 -> xyz=0.020 0 -0.500 rpy=-0.05 0.0 0.0
- joint hip_joint_left: limit lower=-0.5236 upper=0.5236 effort=0 velocity=10.0 -> lower=-1.57 upper=1.57 effort=100 velocity=10.0; origin xyz=0 0.10786 -0.017 rpy=0 0 0 -> xyz=0 0.10786 -0.017 rpy=0 -0.1 0
- joint hip_joint_right: limit lower=-0.5236 upper=0.5236 effort=0 velocity=10.0 -> lower=-1.57 upper=1.57 effort=100 velocity=10.0; origin xyz=0 -0.10786 -0.017 rpy=0 0 0 -> xyz=0 -0.10786 -0.017 rpy=0 0.1 0

Commit message: added arms and hip, need realigned

File: urdf/pady.urdf (robot description, URDF)
Before this commit: robot pady, 7 links, 6 joints
Links:
- added link arm_left, mass 0.150; collision box size=0.261 0.096 0.040; visual mesh filename=package://pady_robot/meshes/visual/arm_left.stl scale=0.001 0.001 0.001
- added link arm_right, mass 0.150; collision box size=0.261 0.096 0.040; visual mesh filename=package://pady_robot/meshes/visual/arm_right.stl scale=0.001 0.001 0.001
Joints:
- added joint arm_joint_left: type revolute, parent base_link, child arm_left, origin xyz=0.100 0.213 -0.017 rpy=0 0 0, axis 0 1 0, limit lower=-1.0 upper=1.0 effort=0 velocity=10.0
- added joint arm_joint_right: type revolute, parent base_link, child arm_right, origin xyz=0.103 -0.293 -0.017 rpy=0 0 0, axis 0 1 0, limit lower=-1.0 upper=1.0 effort=0 velocity=10.0

Commit message: rvis operating, use to move joints to correct location

File: urdf/pady.urdf (robot description, URDF)
Before this commit: robot pady, 9 links, 8 joints
Links:
- link arm_left: geometry collision mesh filename=package://pady_robot/meshes/visual/arm_left.stl scale=0.001 0.001 0.001; visual mesh filename=package://pady_robot/meshes/visual/arm_left.stl scale=0.001 0.001 0.001
- link arm_right: geometry collision mesh filename=package://pady_robot/meshes/visual/arm_right.stl scale=0.001 0.001 0.001; visual mesh filename=package://pady_robot/meshes/visual/arm_right.stl scale=0.001 0.001 0.001
Joints:
- joint arm_joint_right: origin xyz=0.103 -0.293 -0.017 rpy=0 0 0 -> xyz=0.0 -0.26 -0.017 rpy=0 0 0

Commit message: arms and hip fixed, adjusting parameters to achieve 5 consecutive steps

File: urdf/pady.urdf (robot description, URDF)
Before this commit: robot pady, 9 links, 8 joints
Links:
- link arm_left: mass 0.150 -> 0.250
- link arm_right: mass 0.150 -> 0.250
- link foot_left: geometry collision mesh filename=package://pady_robot/meshes/visual/left_foot.stl scale=0.001 0.001 0.001; visual mesh filename=package://pady_robot/meshes/visual/left_foot.stl scale=0.001 0.001 0.001
- link foot_right: geometry collision mesh filename=package://pady_robot/meshes/visual/right_foot.stl scale=0.001 0.001 0.001; visual mesh filename=package://pady_robot/meshes/visual/right_foot.stl scale=0.001 0.001 0.001
Joints:
- joint arm_joint_left: limit lower=-1.0 upper=1.0 effort=0 velocity=10.0 -> lower=-3.14159 upper=3.14159 effort=0 velocity=10.0; origin xyz=0.100 0.213 -0.017 rpy=0 0 0 -> xyz=0.015 0.257 0.008 rpy=0 -1.5708 0
- joint arm_joint_right: limit lower=-1.0 upper=1.0 effort=0 velocity=10.0 -> lower=-3.14159 upper=3.14159 effort=0 velocity=10.0; origin xyz=0.0 -0.26 -0.017 rpy=0 0 0 -> xyz=0.015 -0.26 0.005 rpy=0 -1.5708 0
- joint foot_joint_left: origin xyz=0.020 0 -0.500 rpy=0.05 0.0 0.0 -> xyz=0.020 0 -0.500 rpy=0.0 0.0 0.0
- joint foot_joint_right: origin xyz=0.020 0 -0.500 rpy=-0.05 0.0 0.0 -> xyz=0.020 0 -0.500 rpy=0.0 0.0 0.0
- joint hip_joint_left: limit lower=-1.57 upper=1.57 effort=100 velocity=10.0 -> lower=-0.55 upper=0.55 effort=100 velocity=10.0
- joint hip_joint_right: limit lower=-1.57 upper=1.57 effort=100 velocity=10.0 -> lower=-0.55 upper=0.55 effort=100 velocity=10.0

Commit message: using analysis.launch to find optimal parameters

File: urdf/pady.urdf (robot description, URDF)
Before this commit: robot pady, 9 links, 8 joints
Joints:
- joint arm_joint_left: origin xyz=0.015 0.257 0.008 rpy=0 -1.5708 0 -> xyz=0.015 0.257 0.008 rpy=0 -1.3708 0
- joint arm_joint_right: origin xyz=0.015 -0.26 0.005 rpy=0 -1.5708 0 -> xyz=0.015 -0.26 0.005 rpy=0 -1.7708 0
- joint foot_joint_left: origin xyz=0.020 0 -0.500 rpy=0.0 0.0 0.0 -> xyz=0.020 0 -0.500 rpy=0.1 0.0 0.0
- joint foot_joint_right: origin xyz=0.020 0 -0.500 rpy=0.0 0.0 0.0 -> xyz=0.020 0 -0.500 rpy=-0.1 0.0 0.0
- joint hip_joint_left: limit lower=-0.55 upper=0.55 effort=100 velocity=10.0 -> lower=-0.5760 upper=0.5760 effort=100 velocity=10.0
- joint hip_joint_right: limit lower=-0.55 upper=0.55 effort=100 velocity=10.0 -> lower=-0.5760 upper=0.5760 effort=100 velocity=10.0

Commit message: iterative testing programs

File: urdf/pady.urdf (robot description, URDF)
Before this commit: robot pady, 9 links, 8 joints
Joints:
- joint arm_joint_left: limit lower=-3.14159 upper=3.14159 effort=0 velocity=10.0 -> lower=-1.25 upper=1.25 effort=0 velocity=8.0; origin xyz=0.015 0.257 0.008 rpy=0 -1.5708 0 -> xyz=0.015 0.2585 0.0065 rpy=0 -1.5708 0
- joint arm_joint_right: limit lower=-3.14159 upper=3.14159 effort=0 velocity=10.0 -> lower=-1.25 upper=1.25 effort=0 velocity=8.0; origin xyz=0.015 -0.26 0.005 rpy=0 -1.5708 0 -> xyz=0.015 -0.2585 0.0065 rpy=0 -1.5708 0
- joint foot_joint_left: origin xyz=0.020 0 -0.500 rpy=0.05 0.0 0.0 -> xyz=0.020 0 -0.500 rpy=0.1 0.0 0.0
- joint foot_joint_right: origin xyz=0.020 0 -0.500 rpy=-0.05 0.0 0.0 -> xyz=0.020 0 -0.500 rpy=-0.10 0.0 0.0

Commit message: friday changes

File: urdf/pady.urdf (robot description, URDF)
Before this commit: robot pady, 9 links, 8 joints
Joints:
- joint foot_joint_right: origin xyz=0.020 0 -0.500 rpy=-0.10 0.0 0.0 -> xyz=0.020 0 -0.500 rpy=-0.1 0.0 0.0
- joint hip_joint_left: limit lower=-0.5760 upper=0.5760 effort=100 velocity=10.0 -> lower=-0.5760 upper=0.5760 effort=400 velocity=10.0
- joint hip_joint_right: limit lower=-0.5760 upper=0.5760 effort=100 velocity=10.0 -> lower=-0.5760 upper=0.5760 effort=400 velocity=10.0

Commit message: Update joint limits for thigh joints (33 -. 20 degrees)

File: urdf/pady.urdf (robot description, URDF)
Before this commit: robot pady, 9 links, 8 joints
Joints:
- joint hip_joint_left: limit lower=-0.5760 upper=0.5760 effort=400 velocity=10.0 -> lower=-0.349066 upper=0.349066 effort=400 velocity=10.0
- joint hip_joint_right: limit lower=-0.5760 upper=0.5760 effort=400 velocity=10.0 -> lower=-0.349066 upper=0.349066 effort=400 velocity=10.0

Commit message: configuring walking

File: urdf/pady.urdf (robot description, URDF)
Before this commit: robot pady, 9 links, 8 joints
Links:
- link foot_left: geometry collision cylinder length=0.050 radius=0.008; collision cylinder length=0.050 radius=0.008
- link foot_right: geometry collision cylinder length=0.050 radius=0.008; collision cylinder length=0.050 radius=0.008
Joints:
- joint arm_joint_left: limit lower=-1.25 upper=1.25 effort=0 velocity=8.0 -> lower=-1.53 upper=0.97 effort=0 velocity=8.0; origin xyz=0.015 0.2585 0.0065 rpy=0 -1.5708 0 -> xyz=0.015 0.2585 0.0065 rpy=0 -0.6908 0
- joint arm_joint_right: limit lower=-1.25 upper=1.25 effort=0 velocity=8.0 -> lower=-0.97 upper=1.53 effort=0 velocity=8.0; origin xyz=0.015 -0.2585 0.0065 rpy=0 -1.5708 0 -> xyz=0.015 -0.2585 0.0065 rpy=0 -2.4508 0
- joint foot_joint_left: origin xyz=0.020 0 -0.500 rpy=0.1 0.0 0.0 -> xyz=0.010 0 -0.500 rpy=0.08 0.0 0.0
- joint foot_joint_right: origin xyz=0.020 0 -0.500 rpy=-0.1 0.0 0.0 -> xyz=0.010 0 -0.500 rpy=-0.08 0.0 0.0
- joint hip_joint_left: limit lower=-0.349066 upper=0.349066 effort=400 velocity=10.0 -> lower=-0.0418 upper=0.5418 effort=400 velocity=10.0; origin xyz=0 0.10786 -0.017 rpy=0 -0.1 0 -> xyz=0 0.10786 -0.017 rpy=0 -0.28 0
- joint hip_joint_right: limit lower=-0.349066 upper=0.349066 effort=400 velocity=10.0 -> lower=-0.5418 upper=0.0418 effort=400 velocity=10.0; origin xyz=0 -0.10786 -0.017 rpy=0 0.1 0 -> xyz=0 -0.10786 -0.017 rpy=0 0.28 0
- joint knee_joint_left: limit lower=0.0 upper=1.1345 effort=0 velocity=10.0 -> lower=0.0 upper=1.1345 effort=100 velocity=10.0
- joint knee_joint_right: limit lower=0.0 upper=1.1345 effort=0 velocity=10.0 -> lower=0.0 upper=1.1345 effort=100 velocity=10.0

Commit message: robot one step potentail for more

File: urdf/pady.urdf (robot description, URDF)
Before this commit: robot pady, 9 links, 8 joints
Links:
- link foot_left: geometry collision mesh filename=package://pady_robot/meshes/visual/left_foot.stl scale=0.001 0.001 0.001; visual mesh filename=package://pady_robot/meshes/visual/left_foot.stl scale=0.001 0.001 0.001
- link foot_right: geometry collision mesh filename=package://pady_robot/meshes/visual/right_foot.stl scale=0.001 0.001 0.001; visual mesh filename=package://pady_robot/meshes/visual/right_foot.stl scale=0.001 0.001 0.001
Joints:
- joint foot_joint_left: origin xyz=0.010 0 -0.500 rpy=0.08 0.0 0.0 -> xyz=0.0 0 -0.500 rpy=0.08 0.0 0.0
- joint foot_joint_right: origin xyz=0.010 0 -0.500 rpy=-0.08 0.0 0.0 -> xyz=0.0 0 -0.500 rpy=-0.08 0.0 0.0

Commit message: robot most stable, fix foot pivoting only

File: urdf/pady.urdf (robot description, URDF)
Before this commit: robot pady, 9 links, 8 joints
Links:
- link arm_left: geometry visual mesh filename=package://pady_robot/meshes/visual/arm_left.stl scale=0.001 0.001 0.001
- link arm_right: geometry visual mesh filename=package://pady_robot/meshes/visual/arm_right.stl scale=0.001 0.001 0.001

Commit message: yaw reducing script works, 3 steps achieved, start plotting data

File: urdf/pady.urdf (robot description, URDF)
Before this commit: robot pady, 9 links, 8 joints
Links:
- added link yaw_anchor, mass 0.0001
- link arm_left: mass 0.250 -> 0.300
- link arm_right: mass 0.250 -> 0.300
Joints:
- added joint yaw_joint: type revolute, parent yaw_anchor, child base_link, axis 0 0 1, limit lower=-3.14159 upper=3.14159 effort=100 velocity=10.0

Commit message: video evidence

File: urdf/pady.urdf (robot description, URDF)
Before this commit: robot pady, 10 links, 9 joints
Links:
- link arm_left: geometry collision mesh filename=package://pady_robot/meshes/visual/arm_left.stl scale=0.001 0.001 0.001; visual mesh filename=package://pady_robot/meshes/visual/arm_left.stl scale=0.001 0.001 0.001
- link arm_right: geometry collision mesh filename=package://pady_robot/meshes/visual/arm_right.stl scale=0.001 0.001 0.001; visual mesh filename=package://pady_robot/meshes/visual/arm_right.stl scale=0.001 0.001 0.001
